Commit message: Succcessful Pick and Place and Added Grasp Fix Plugin

File: xarm_ros2/xarm_description/urdf/gripper/xarm_gripper.gazebo.xacro (robot description, xacro)
@@ -35,22 +35,19 @@
     </gazebo>
   </xacro:macro>
-  <xacro:macro name="xarm_gazebo_grasp_fix" params="prefix:='' arm_name:='xarm_gripper' palm_link:='link_base'">
+  <xacro:macro name="xarm_gazebo_grasp_fix" params="prefix:='' arm_name:='xarm7' palm_link:='link7'">
     <gazebo>
       <plugin name="gazebo_grasp_fix" filename="libgazebo_grasp_fix.so">
         <arm>
-          <arm_name>${arm_name}</arm_name>
-          <palm_link>${palm_link}</palm_link>
+          <arm_name>xarm7</arm_name>
+          <palm_link>${prefix}link7</palm_link> <gripper_link>${prefix}left_finger</gripper_link>
+          <gripper_link>${prefix}right_finger</gripper_link>
           <gripper_link>${prefix}left_inner_knuckle</gripper_link>
           <gripper_link>${prefix}right_inner_knuckle</gripper_link>
-          <!-- <gripper_link>${prefix}left_outer_knuckle</gripper_link>
-          <gripper_link>${prefix}right_outer_knuckle</gripper_link> -->
-          <gripper_link>${prefix}left_finger</gripper_link>
-          <gripper_link>${prefix}right_finger</gripper_link>
         </arm>
         <forces_angle_tolerance>100</forces_angle_tolerance>
-        <update_rate>10</update_rate>
-        <grip_count_threshold>2</grip_count_threshold>
-        <max_grip_count>3</max_grip_count>
-        <release_tolerance>0.0198</release_tolerance>
+        <update_rate>30</update_rate>
+        <grip_count_threshold>1</grip_count_threshold>
+        <max_grip_count>2</max_grip_count>
+        <release_tolerance>0.005</release_tolerance>
         <disable_collisions_on_attach>false</disable_collisions_on_attach>
         <contact_topic>__default_topic__</contact_topic>
