Commit message: Made the workpiece to be in-front to solve weird solutions of IK solver

File: xarm_ros2/xarm_moveit_config/srdf/_xarm7_macro.srdf.xacro (robot description, xacro)
@@ -46,5 +46,5 @@
       <joint name="${prefix}joint4" value="0" />
       <joint name="${prefix}joint5" value="0" />
-      <joint name="${prefix}joint6" value="0" />
+      <joint name="${prefix}joint6" value="-1.5708" />
       <joint name="${prefix}joint7" value="0" />
     </group_state>
